File: logic-lp384/prj-kicad/pmod-logic-lp384.sch (KiCad schematic (older format))
At the start: 3 parts, among them P1 PMOD, U1 ICE40LP384-SG32

Commit message: Logic-LP384: Update schematics
Parts:
- removed P?: PMOD, symbol PMOD
- added C1: 1uF, pmod-logic-lp384:SMD0805, symbol C
- added C10, C2: 1uF, pmod-logic-lp384:SMD0603, symbol C
- added C3, C5, C9: 4.7uF, pmod-logic-lp384:SMD0603, symbol C
- added C4: 100nF, pmod-logic-lp384:SMD0603, symbol C
- added C6, C7: C, pmod-logic-lp384:SMD0603, symbol C
- added C8: 10uF, pmod-logic-lp384:SMD0805, symbol C
- added L1: 2.2uH, pmod-logic-lp384:SMD0603, symbol INDUCTOR
- added P2: PMOD, pmod-logic-lp384:PMOD_SSW106-RA, symbol PMOD
- added P3: JUMPER, pmod-logic-lp384:CONN_2, symbol JUMPER
- added P4: CONN_6, pmod-logic-lp384:CONN_6, symbol CONN_6
- added U2: TXS0108E-PW, pmod-logic-lp384:TSSOP20, symbol TXS0108E-PW
- added U3: LM3671, pmod-logic-lp384:SOT23-5, symbol LM3671
- added U4: TPS763xx, pmod-logic-lp384:SOT23-5, symbol TPS763xx
- added U5: SST25VF, pmod-logic-lp384:SMD_SO8E, symbol SST25VF
- P1: footprint (none) -> pmod-logic-lp384:CONN_PMOD-Male
- U1: footprint (none) -> pmod-logic-lp384:QFN32
Connections:
- net DATA_6: now reaches U1.1 (IOL_2B)
- net DATA_6: now also U2.7 (A6)
- net SPI_SDO: now reaches U1.12 (IOB_24_SDO)
- net SPI_SDO: now also P4.2 (P2), U5.2 (DO)
- net SPI_SDI: now reaches U1.13 (IOB_25_SDI)
- net SPI_SDI: now also P4.4, U5.5 (DI)
- net SPI_SS: now reaches U1.14 (IOB_27_SS)
- net SPI_SS: now also P4.3 (P3), U5.1 (CS)
- net SPI_SCK: now reaches U1.15 (IOB_26_SCK)
- net SPI_SCK: now also P4.6, U5.6 (CLK)
- net IN_1: now reaches U1.18 (IOR_34)
- net IN_1: now also P1.1 (IO1)
- net IN_5: now reaches U1.19 (IOR_35)
- net IN_5: now also P1.7 (IO5)
- net DATA_5: now reaches U1.2 (IOL_2A)
- net DATA_5: now also U2.6 (A5)
- net IN_2: now reaches U1.20 (IOR_36)
- net IN_2: now also P1.2 (IO2)
- net IN_6: now reaches U1.22 (IOR_38)
- net IN_6: now also P1.8 (IO6)
- net IN_3: now reaches U1.23 (IOR_39)
- net IN_3: now also P1.3 (IO3)
- net IN_8: now reaches U1.26 (IOT_45)
- net IN_8: now also P1.10 (IO8)
- net IN_4: now reaches U1.27 (IOT_47)
- net IN_4: now also P1.4 (IO4)
- net IN_7: now reaches U1.29 (IOT_49)
- net IN_7: now also P1.9 (IO7)
- net DATA_OE: now reaches U1.30 (IOT_50)
- net DATA_OE: now also U2.10 (OE)
- net DATA_8: now reaches U1.31 (IOT_53)
- net DATA_8: now also U2.9 (A8)
- net DATA_7: now reaches U1.32 (IOT_52)
- net DATA_7: now also U2.8 (A7)
- net DATA_4: now reaches U1.5 (IOL_4A)
- net DATA_4: now also U2.5 (A4)
- net DATA_3: now reaches U1.6 (IOL_4B)
- net DATA_3: now also U2.4 (A3)
- net DATA_2: now reaches U1.7 (IOL_5B)
- net DATA_2: now also U2.3 (A2)
- net DATA_1: now reaches U1.8 (IOL_5A)
- net DATA_1: now also U2.1 (A1)
- net GND: now reaches P1.11
- net GND: now also P1.5, U1.21, U1.3, C1.2, C10.2, C2.2, C3.2, C4.2, C5.2, C6.2, C7.2, C8.2, C9.2, P2.11, P2.5, P4.1 (P1), U2.11, U3.2, U4.2, U5.4
- net +3.3V: now reaches P1.12
- net +3.3V: now also P1.6, U1.16 (V_SPI), U1.17 (VIO_1), U1.28 (VIO_0), U1.4 (VIO_3), U1.9 (VIO_2), C1.1, C10.1, C2.1, C4.1, C8.1, C9.1, P3.1, U2.2 (VCCA), U3.1 (VIN), U3.3 (EN), U4.1 (VIN), U4.3 (EN), U5.3 (WP), U5.7 (HOLD), U5.8
- net RST: now reaches U1.10 (Reset)
- net RST: now also P4.5
- net +2.5V: now reaches U1.24 (VPP)
- net +2.5V: now also C5.1, U4.5 (Vout)
- net +1.2V: now reaches U1.25 (VCC)
- net +1.2V: now also C3.1, L1.2, U3.4 (FB)
- new net: L1.1, U3.5 (SW)
- new net +Vcc: C6.1, C7.1, P2.12, P2.6, P3.2, U2.19 (VCCB)
- new net OUT_1: P2.1 (IO1), U2.20 (B1)
- new net OUT_2: P2.2 (IO2), U2.17 (B3)
- new net OUT_3: P2.3 (IO3), U2.15 (B5)
- new net OUT_4: P2.4 (IO4), U2.13 (B7)
- new net OUT_5: P2.7 (IO5), U2.18 (B2)
- new net OUT_6: P2.8 (IO6), U2.16 (B4)
- new net OUT_7: P2.9 (IO7), U2.14 (B6)
- new net OUT_8: P2.10 (IO8), U2.12 (B8)
- no-connect marks 0 -> 2
Other:
- note added: "PLD / Internal logic"
- note added: "PLD Memory"
- note added: "PMOD Inputs"
- note added: "PMOD Outputs"
- note added: "Power Supply"
